File: X4/MSX_Expander_X4.kicad_sch (KiCad schematic)
At the start: 21 parts, among them J1 IDC50P - MSX BUS, J2 MSX SLOT CONNECTOR 0, J3 MSX SLOT CONNECTOR 1, U1 74LS273, U2 74LS540, U3 74LS352, U4 74LS139, U5 74LS11, U6 74LS133, U7 74LS32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

Commit message: routing pcb
Parts:
- removed C4, C5, C6, C7, C8: 0.1, Capacitors_THT:C_Disc_D4.7mm_W2.5mm_P5.00mm, symbol MSXIOSlot-rescue:C_Small
- removed U1: 74LS273, symbol 74xx:74LS273
- removed U2: 74LS540, symbol 74xx:74LS540
- removed U3: 74LS352, symbol 74xx:74LS352
- removed U4: 74LS139, symbol 74xx_IEEE:74LS139
- removed U6: 74LS133, symbol 74xx:74LS133
- removed unit 1 of U7
- C1, C2, C3: footprint Capacitors_THT:C_Disc_D4.7mm_W2.5mm_P5.00mm -> Capacitor_THT:C_Disc_D5.0mm_W2.5mm_P5.00mm
- J1: footprint Roni Footprints:IDC-Header_2x25_P2.54mm_Vertical -> Connector_IDC:IDC-Header_2x25_P2.54mm_Vertical
- J2: value MSX SLOT CONNECTOR 0 -> MSX SUB-SLOT 0; footprint Roni Footprints:IDC-Header_2x25_P2.54mm_Vertical -> Roni Footprints:50_pin_edge_female
- J3: value MSX SLOT CONNECTOR 1 -> MSX SUB-SLOT 1; footprint Roni Footprints:IDC-Header_2x25_P2.54mm_Vertical -> Roni Footprints:50_pin_edge_female
- U5, U7, U9: footprint (none) -> Package_DIP:DIP-14_W7.62mm
Connections:
- net A10: no longer U5.1
- net A11: no longer U5.2
- net A12: no longer U5.13
- net A13: no longer U5.3
- net A14: no longer U5.4
- net A15: no longer U5.5
- net EXP_SLTSL0: now also J1.5 (Pin_5)
- net EXP_SLTSL1: now also J1.16 (Pin_16)
- net SOUNDIN: no longer J2.49 (Pin_49), J3.49 (Pin_49)
- net at U5.6: no longer U5.12
- net SOUND_A renamed SOUND0
- net SOUND0: now also J2.49 (Pin_49)
- net SOUND_B renamed SOUND1
- net SOUND1: now also J3.49 (Pin_49)
- no-connect marks 18 -> 23
Other:
- moved on the sheet: J1, J2, J3, R8, R9
