File: X4/MSX_Expander_X4_Cart.kicad_sch (KiCad schematic)
At the start: 17 parts, among them J1 MSX Edge Connector, J2 IDC50P - MSX BUS, U1 74LS273, U2 74LS540, U3 74LS352, U4 74LS139, U5 74LS11, U6 74LS133, U7 74LS32

Commit message: started routing
Parts:
- added unit 2 of U6
- J1: footprint Roni Footprints:MSX_CART_SW -> Roni Footprints:MSX_CART_SW_Official
Connections:
- net +5V: now also U6.16 (VCC)
- net GND: now also U6.8 (GND)
Changed lines of the file:
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@@
     (property "Reference" "J1" (id 0) (at 222.885 29.845 0))
     (property "Value" "MSX Edge Connector" (id 1) (at 222.885 33.02 0))
-    (property "Footprint" "Roni Footprints:MSX_CART_SW" (id 2) (at 222.885 68.58 0)
+    (property "Footprint" "Roni Footprints:MSX_CART_SW_Official" (id 2) (at 222.885 68.58 0)
       (effects (font (size 1.27 1.27)) hide)
     )
@@
     (pin "1")
   )
+  (symbol (lib_id "74xx:74LS133") (at 92.71 262.255 0) (unit 2)
+    (in_bom yes) (on_board yes)
+    (property "Reference" "U6" (id 0) (at 90.805 262.255 0)
+      (effects (font (size 1.27 1.27)) (justify left))
+    )
+    (property "Value" "74LS133" (id 1) (at 93.345 252.73 0)
+      (effects (font (size 1.27 1.27)) (justify left))
+    )
+    (property "Footprint" "Package_DIP:DIP-16_W7.62mm" (id 2) (at 92.71 262.255 0)
+      (effects (font (size 1.27 1.27)) hide)
+    )
+    (property "Datasheet" "http://www.ti.com/lit/gpn/sn74LS133" (id 3) (at 92.71 262.255 0)
+      (effects (font (size 1.27 1.27)) hide)
+    )
+    (pin "1")
+    (pin "10")
+    (pin "11")
+    (pin "12")
+    (pin "13")
+    (pin "14")
+    (pin "15")
+    (pin "2")
+    (pin "3")
+    (pin "4")
+    (pin "5")
+    (pin "6")
+    (pin "7")
+    (pin "9")
+    (pin "16")
+    (pin "8")
+  )
   (symbol (lib_id "power:GND") (at 182.245 154.94 0) (unit 1)
     (in_bom yes) (on_board yes)
@@
     (pin "1")
   )
+  (symbol (lib_id "power:GND") (at 92.71 274.955 0) (unit 1)
+    (in_bom yes) (on_board yes)
+    (property "Reference" "#PWR0109" (id 0) (at 92.71 281.305 0)
+      (effects (font (size 1.27 1.27)) hide)
+    )
+    (property "Value" "GND" (id 1) (at 92.71 278.765 0)
+      (effects (font (size 1 1)))
+    )
+    (property "Footprint" "" (id 2) (at 92.71 274.955 0)
+      (effects (font (size 1.27 1.27)) hide)
+    )
+    (property "Datasheet" "" (id 3) (at 92.71 274.955 0)
+      (effects (font (size 1.27 1.27)) hide)
+    )
+    (pin "1")
+  )
   (symbol (lib_id "power:+5V") (at 69.215 249.555 0) (unit 1)
     (in_bom yes) (on_board yes) (fields_autoplaced)
@@
     (pin "7")
   )
+  (symbol (lib_id "power:+5V") (at 92.71 249.555 0) (unit 1)
+    (in_bom yes) (on_board yes) (fields_autoplaced)
+    (property "Reference" "#PWR0110" (id 0) (at 92.71 253.365 0)
+      (effects (font (size 1.27 1.27)) hide)
+    )
+    (property "Value" "+5V" (id 1) (at 92.71 243.84 0))
+    (property "Footprint" "" (id 2) (at 92.71 249.555 0)
+      (effects (font (size 1.27 1.27)) hide)
+    )
+    (property "Datasheet" "" (id 3) (at 92.71 249.555 0)
+      (effects (font (size 1.27 1.27)) hide)
+    )
+    (pin "1")
+  )
   (symbol (lib_id "74xx:74LS11") (at 75.565 65.405 0) (unit 1)
     (in_bom yes) (on_board yes)
@@
       (reference "#PWR0108") (unit 1) (value "+5V") (footprint "")
     )
+    (path "/c704f1f0-32ac-4340-8574-ec31bafab5c3"
+      (reference "#PWR0109") (unit 1) (value "GND") (footprint "")
+    )
+    (path "/eeb188c4-356a-42f6-873b-da2b33ead2b6"
+      (reference "#PWR0110") (unit 1) (value "+5V") (footprint "")
+    )
     (path "/9d013d68-611e-44e2-b024-6e1bbf371fa8"
       (reference "#PWR0111") (unit 1) (value "GND") (footprint "")
@@
     )
     (path "/00000000-0000-0000-0000-00005a85a267"
-      (reference "J1") (unit 1) (value "MSX Edge Connector") (footprint "Roni Footprints:MSX_CART_SW")
+      (reference "J1") (unit 1) (value "MSX Edge Connector") (footprint "Roni Footprints:MSX_CART_SW_Official")
     )
     (path "/2766d971-d226-499a-b67f-0ce3b8285b78"
@@
       (reference "U6") (unit 1) (value "74LS133") (footprint "Package_DIP:DIP-16_W7.62mm")
     )
+    (path "/65783835-2c2e-4a0a-ad68-d242ff77951c"
+      (reference "U6") (unit 2) (value "74LS133") (footprint "Package_DIP:DIP-16_W7.62mm")
+    )
     (path "/edd189ed-8849-405c-98d6-8ada54dea003"
